File: OpenC16Cart.kicad_pcb (KiCad board)
At the start: 2 copper layers, 52 x 65 mm, 16 parts, among them J1 CONN_02X03, J11 CONN_01X03, J12 CONN_01X03, J2 CONN_01X03, J21 CONN_01X03, J22 CONN_01X03, J3 CONN_01X03, J4 CONN_02X03, J5 CONN_01X03, J6 CONN_01X03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

Commit message: Bump version
Other:
- board text added: "V3"
- board text removed: "V2"
Changed lines of the file:
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@@
   (gr_arc (start 172 127) (end 173.5 127) (angle 90) (layer Edge.Cuts) (width 0.15))
   (gr_arc (start 123 127) (end 123 128.5) (angle 90) (layer Edge.Cuts) (width 0.15))
-  (gr_text V2 (at 124.46 118.872) (layer B.SilkS)
+  (gr_text V3 (at 124.46 118.872) (layer B.SilkS)
     (effects (font (size 1 1) (thickness 0.2)) (justify mirror))
   )

Commit message: Minor tweaks'n'fixes
Parts:
- J1, J4: footprint Pin_Headers:Pin_Header_Straight_2x03_Pitch2.54mm -> OpenC16Cart:Pin_Header_Straight_2x03-ModSilkS
- J11, J12, J2, J21, J22, J3, J5, J6: footprint Pin_Headers:Pin_Header_Straight_1x03_Pitch2.54mm -> OpenC16Cart:Pin_Header_Straight_1x03-ModSilkS
- J7: footprint C16_Cart_Conn:C16_Cart_Conn -> OpenC16Cart:C16_Cart_Conn
- U1, U2: footprint C16_Cart_Conn:dil_28-600_socket_ThinSilkS -> OpenC16Cart:dil_28-600_socket_ThinSilkS
Connections:
- J7 pad 10: Net-(J7-Pad10) -> (no net)
- J7 pad 11: Net-(J7-Pad11) -> (no net)
- J7 pad 12: Net-(J7-Pad12) -> (no net)
- J7 pad 13: Net-(J7-Pad13) -> (no net)
- J7 pad 22: Net-(J7-Pad22) -> (no net)
- J7 pad 23: Net-(J7-Pad23) -> (no net)
- J7 pad 24: Net-(J7-Pad24) -> (no net)
- J7 pad 4: Net-(J7-Pad4) -> (no net)
- J7 pad 5: Net-(J7-Pad5) -> (no net)
- J7 pad 7: Net-(J7-Pad7) -> (no net)
- J7 pad 8: Net-(J7-Pad8) -> (no net)
- J7 pad 9: Net-(J7-Pad9) -> (no net)
- J7 pad AA: Net-(J7-PadAA) -> (no net)
- J7 pad BB: Net-(J7-PadBB) -> (no net)
- J7 pad C: Net-(J7-PadC) -> (no net)
- J7 pad D: Net-(J7-PadD) -> (no net)
- J7 pad E: Net-(J7-PadE) -> (no net)
- J7 pad F: Net-(J7-PadF) -> (no net)
- J7 pad H: Net-(J7-PadH) -> (no net)
- J7 pad Z: Net-(J7-PadZ) -> (no net)
Routing:
- net /a12: track 138.9 -> 136.6 mm
- net VCC: track 150.2 -> 149.3 mm

Commit message: Final touches for V3
Parts:
- moved J7 0.05 mm to (147.5, 124.5)

Commit message: Much better
Parts:
- removed G***: LOGO, w_logo:Logo_copper_OSHW_6x6mm
- removed J2, J3, J5, J6: CONN_01X03, OpenC16Cart:Pin_Header_Straight_1x03-ModSilkS
- removed J7: C16-Exp-Port, OpenC16Cart:C16_Cart_Conn
- added CN1: C16-Exp-Port, OpenC16Cart:C16_Cart_Conn, F.Cu at (147.5, 124.5)
- added H1: MountingHole, MountingHole:MountingHole_3.2mm_M3, F.Cu at (147.5, 72.1)
- added V0: LICENSE, OpenC16Cart:cc_by_nc_sa, B.Cu at (142.4, 115.6)
- C1, C2: value C -> 100n; footprint Capacitors_SMD:C_0805_HandSoldering -> Capacitor_THT:C_Disc_D7.0mm_W2.5mm_P5.00mm
- J1, J4: value CONN_02X03 -> Conn_02x03_Odd_Even; footprint OpenC16Cart:Pin_Header_Straight_2x03-ModSilkS -> Connector_PinHeader_2.54mm:PinHeader_2x03_P2.54mm_Vertical
- J11, J12, J21, J22: value CONN_01X03 -> Conn_01x03_Male; footprint OpenC16Cart:Pin_Header_Straight_1x03-ModSilkS -> Connector_PinHeader_2.54mm:PinHeader_1x03_P2.54mm_Vertical
- U1, U2: footprint OpenC16Cart:dil_28-600_socket_ThinSilkS -> Package_DIP:DIP-28_W15.24mm_Socket_LongPads
- moved U2 18.1 mm to (167.5, 110.5), turned to 180 degrees
- moved U1 17.4 mm to (142.7, 110.5), turned to 180 degrees
- moved C2 5.98 mm to (152.3, 114.3), turned to 0 degrees
- moved J11 5.58 mm to (136.4, 67.1)
- moved C1 5.23 mm to (127.5, 114.3), turned to 0 degrees
- moved J12 4.19 mm to (141.4, 67.1)
- moved J21 3.68 mm to (161.2, 67.1)
- moved J22 2.29 mm to (166.1, 67.1)
- moved J4 2.03 mm to (153.7, 67.1)
- moved J1 0.13 mm to (128.9, 67.1)
Connections:
- C1 pad 1: GND -> VCC
- C1 pad 2: VCC -> GND
- C2 pad 1: GND -> VCC
- C2 pad 2: VCC -> GND
- U1 pad 20: //ce_u1 -> GND
- U1 pad 22: Net-(J7-PadB) -> /~c1lo
- U1 pad 23: /a11_u1 -> /a11
- U2 pad 20: //ce_u2 -> GND
- U2 pad 22: Net-(J7-Pad6) -> /~c1hi
- U2 pad 23: /a11_u2 -> /a11
Routing:
- net /a11_conn: track 98.1 -> 0.00 mm, vias 1 -> 0
- net /a12: track 136.6 -> 54.4 mm
- net /~c1hi: track 0.00 -> 59.2 mm, vias 0 -> 2
- net /a11: track 0.00 -> 54.9 mm, vias 0 -> 1
- net Net-(J7-Pad6): track 49.6 -> 0.00 mm, vias 1 -> 0
- net /a11_u1: track 49.5 -> 0.00 mm
- net //ce_u1: track 46.5 -> 0.00 mm
- net /~c1lo: track 0.00 -> 43.8 mm, vias 0 -> 1
- net /a11_u2: track 41.0 -> 0.00 mm
- net Net-(J7-PadB): track 33.2 -> 0.00 mm
- net //ce_u2: track 32.9 -> 0.00 mm
- net /a14_u2: track 65.3 -> 44.9 mm, vias 0 -> 1
- net VCC: track 149.3 -> 132.3 mm, vias 1 -> 0
- net GND: track 145.0 -> 133.1 mm
- net /d7: track 67.1 -> 78.2 mm, vias 1 -> 2
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Other:
- net class Default: clearance 0.25 -> 0.2; trace_width 0.254 -> 0.25; via_dia 1 -> 0.6; via_drill 0.5 -> 0.4
- net class Power: clearance 0.254 -> 0.2; trace_width 0.508 -> 0.5; via_dia 1.4 -> 0.8; via_drill 0.8 -> 0.6
- rule trace_clearance: 0.25 -> 0.2
- rule via_min_size: 0.6 -> 0.4
- board text added: "A13"
- board text added: "CC-BY-NC-SA © SukkoPera 2017-2023 github.com/SukkoPera/OpenC16Cart"
- board text added: "V4"
- board text removed: "J1/A13"
- board text removed: "J4/A13"
- board text removed: "V3"
- board text removed: "github.com/SukkoPera/OpenC16Cart"
